File: matrix.sch (KiCad schematic (older format))
At the start: 124 parts, among them K1 KEYSW, K10 KEYSW, K11 KEYSW, K12 KEYSW, K13 KEYSW, K14 KEYSW, K15 KEYSW, K16 KEYSW, K17 KEYSW, K18 KEYSW, K19 KEYSW, K2 KEYSW, K20 KEYSW, K21 KEYSW, K22 KEYSW, K23 KEYSW, K24 KEYSW, K25 KEYSW, K26 KEYSW, K27 KEYSW, K28 KEYSW, K29 KEYSW, K3 KEYSW, K30 KEYSW, K31 KEYSW, K32 KEYSW, K33 KEYSW, K34 KEYSW, K35 KEYSW, K36 KEYSW, K37 KEYSW, K38 KEYSW, K39 KEYSW, K4 KEYSW, K40 KEYSW, K42 KEYSW, K43 KEYSW, K45 KEYSW, K46 KEYSW, K47 KEYSW, K48 KEYSW, K49 KEYSW, K5 KEYSW, K50 KEYSW, K51 KEYSW, K52 KEYSW, K53 KEYSW, K54 KEYSW, K56 KEYSW, K57 KEYSW, K58 KEYSW, K59 KEYSW, K6 KEYSW, K60 KEYSW, K62 KEYSW, K63 KEYSW, K64 KEYSW, K65 KEYSW, K7 KEYSW, K8 KEYSW, K9 KEYSW

Commit message: Add files via upload
Other:
- moved on the sheet: D1, D10, D11, D12, D13, D14, D15, D16, D17, D18, D19, D2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

Commit message: Add files via upload
Parts:
- renumbered R4 to R6
Changed lines of the file:
@@
 LIBS:zetex
 LIBS:Zilog
+LIBS:IS31FL3236-QFLS2-TR
+LIBS:teensy
+LIBS:IS31FL37XX
+LIBS:crumpschemes
+LIBS:led
 LIBS:Poliboard3-cache
 EELAYER 25 0
@@
 extra1
 $Comp
-L VCC #PWR08
+L VCC #PWR017
 U 1 1 59996913
 P 7850 8700
-F 0 "#PWR08" H 7850 8550 50  0001 C CNN
+F 0 "#PWR017" H 7850 8550 50  0001 C CNN
 F 1 "VCC" H 7850 8850 50  0000 C CNN
 F 2 "" H 7850 8700 50  0001 C CNN
@@
 $EndComp
 $Comp
-L R R4
+L R R6
 U 1 1 59998030
 P 8200 9350
-F 0 "R4" V 8280 9350 50  0000 C CNN
+F 0 "R6" V 8280 9350 50  0000 C CNN
 F 1 "300" V 8200 9350 50  0000 C CNN
 F 2 "Resistors_SMD:R_0805_HandSoldering" V 8130 9350 50  0001 C CNN
