File: Charlieplex LED.sch (KiCad schematic (older format))
At the start: 77 parts

Commit message: Add files via upload
Connections:
- net CA5: no longer DB13.1 (A), DB21.1 (A), DB29.1 (A), DB37.1 (A), DB41.2 (K), DB42.2 (K), DB43.2 (K), DB44.2 (K), DB45.2 (K), DB46.2 (K), DB47.2 (K), DB48.2 (K), DB5.1 (A), DB54.1 (A)
- net CA6: now also DB13.1 (A), DB21.1 (A), DB29.1 (A), DB37.1 (A), DB41.2 (K), DB42.2 (K), DB43.2 (K), DB44.2 (K), DB45.2 (K), DB46.2 (K), DB47.2 (K), DB48.2 (K), DB5.1 (A), DB54.1 (A); no longer DB14.1 (A), DB22.1 (A), DB30.1 (A), DB38.1 (A), DB46.1 (A), DB49.2 (K), DB50.2 (K), DB51.2 (K), DB52.2 (K), DB53.2 (K), DB54.2 (K), DB55.2 (K), DB56.2 (K), DB6.1 (A)
- net CA7: now also DB14.1 (A), DB22.1 (A), DB30.1 (A), DB38.1 (A), DB46.1 (A), DB49.2 (K), DB50.2 (K), DB51.2 (K), DB52.2 (K), DB53.2 (K), DB54.2 (K), DB55.2 (K), DB56.2 (K), DB6.1 (A); no longer DB15.1 (A), DB16.1 (A), DB23.1 (A), DB24.1 (A), DB31.1 (A), DB32.1 (A), DB39.1 (A), DB40.1 (A), DB47.1 (A), DB48.1 (A), DB55.1 (A), DB56.1 (A), DB57.2 (K), DB58.2 (K), DB59.2 (K), DB60.2 (K), DB61.2 (K), DB7.1 (A), DB8.1 (A)
- new net CA8: DB15.1 (A), DB16.1 (A), DB23.1 (A), DB24.1 (A), DB31.1 (A), DB32.1 (A), DB39.1 (A), DB40.1 (A), DB47.1 (A), DB48.1 (A), DB55.1 (A), DB56.1 (A), DB57.2 (K), DB58.2 (K), DB59.2 (K), DB60.2 (K), DB61.2 (K), DB7.1 (A), DB8.1 (A)
Other:
- note added: "B62"
- note added: "B63\n"
- note added: "B64"
- note added: "B65"
- note added: "B66"
- note added: "B67"
- note added: "B68"
- note added: "B69\n"
- note added: "B70"
- note added: "B71"
- note added: "B72"
- note added: "B73\n"
- note added: "B74"
- note added: "B75"
- note added: "B76"
- note added: "B77\n"
- note added: "G62"
- note added: "G63\n"
- note added: "G64"
- note added: "G65"
- note added: "G66"
- note added: "G67"
- note added: "G68"
- note added: "G69"
- note added: "G70"
- note added: "G71"
- note added: "G72"
- note added: "G73"
- note added: "G74"
- note added: "G75"
- note added: "G76"
- note added: "G77"
- note added: "R62"
- note added: "R63"
- note added: "R64"
- note added: "R65"
- note added: "R66"
- note added: "R67"
- note added: "R68"
- note added: "R69"
- note added: "R70"
- note added: "R71"
- note added: "R72"
- note added: "R73"
- note added: "R74"
- note added: "R75"
- note added: "R76"
- note added: "R77"
- moved on the sheet: DB1, DB10, DB11, DB12, DB13, DB14, DB15, DB16, DB17, DB18, DB19, DB2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
