File: Poliboard3.kicad_pcb (KiCad board)
At the start: 2 copper layers, 285.8 x 95.3 mm, 242 parts, among them K1 KEYSW, K10 KEYSW, K11 KEYSW, K12 KEYSW, K13 KEYSW, K14 KEYSW, K15 KEYSW, K16 KEYSW, K17 KEYSW, K18 KEYSW, K19 KEYSW, K2 KEYSW, K20 KEYSW, K21 KEYSW, K22 KEYSW, K23 KEYSW, K24 KEYSW, K25 KEYSW, K26 KEYSW, K27 KEYSW, K28 KEYSW, K29 KEYSW, K3 KEYSW, K30 KEYSW, K31 KEYSW, K32 KEYSW, K33 KEYSW, K34 KEYSW, K35 KEYSW, K36 KEYSW, K37 KEYSW, K38 KEYSW, K39 KEYSW, K4 KEYSW, K40 KEYSW, K42 KEYSW, K43 KEYSW, K45 KEYSW, K46 KEYSW, K47 KEYSW, K48 KEYSW, K49 KEYSW, K5 KEYSW, K50 KEYSW, K51 KEYSW, K52 KEYSW, K53 KEYSW, K54 KEYSW, K56 KEYSW, K57 KEYSW, K58 KEYSW, K59 KEYSW, K6 KEYSW, K60 KEYSW, K62 KEYSW, K63 KEYSW, K64 KEYSW, K65 KEYSW, K7 KEYSW, K8 KEYSW, K9 KEYSW, P0 CONN_1, P01 CONN_1, P02 CONN_1, P1 CONN_1, P10 CONN_1, P11 CONN_1, P12 CONN_1, P13 CONN_1, P14 CONN_1, P15 CONN_1, P16 CONN_1, P17 CONN_1, P18 CONN_1, P19 CONN_1, P2 CONN_1, P20 CONN_1, P21 CONN_1, P22 CONN_1, P23 CONN_1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

Commit message: Add files via upload
Parts:
- removed DB62, DB63, DB64, DB65: LED, mx1a:MX1A-led_no3d
- removed P0, P01, P02, P10, P11, P12, P13, P14, P15, P16, P17, P18, P19, P20, P21, P22, P23, P24, P25, P26, P27, P28, P29, P30, P31, P32, P33, P34, P35, P36, P37, P38, P39, P40, P41, P42, P43, P5, P6, P7, P8, P9: CONN_1, Custom:CONN_1
- added C1: 1u, Capacitors_SMD:C_0805_HandSoldering, B.Cu at (188.1, 166.7)
- added DB41: LED, mx1a:MX1A-led_no3d, F.Cu at (338.1, 126.2)
- added DB44: LED, mx1a:MX1A-led_no3d, F.Cu at (145.3, 145.3)
- added DB55: LED, mx1a:MX1A-led_no3d, F.Cu at (109.5, 164.3)
- added DB61: LED, mx1a:MX1A-led_no3d, F.Cu at (347.7, 164.3)
- added GND1: CONN_1, keyboard_parts:PIN_1, F.Cu at (228.6, 164.3)
- added GND2: CONN_1, keyboard_parts:PIN_1, F.Cu at (119.1, 100.0)
- added GND3: CONN_1, keyboard_parts:PIN_1, F.Cu at (114.3, 140.5)
- added GND4: CONN_1, keyboard_parts:PIN_1, F.Cu at (314.3, 147.6)
- added GND5: CONN_1, keyboard_parts:PIN_1, F.Cu at (269.1, 109.5)
- added LED62: LED-RGB-CA, LEDs:LED_D5.0mm-4, B.Cu at (78.6, 109.5)
- added LED63: LED-RGB-CA, LEDs:LED_D5.0mm-4, B.Cu at (78.6, 142.9)
- added LED64: LED-RGB-CA, LEDs:LED_D5.0mm-4, B.Cu at (109.5, 81.0)
- added LED65: LED-RGB-CA, LEDs:LED_D5.0mm-4, B.Cu at (100.0, 169.1)
- added LED66: LED-RGB-CA, LEDs:LED_D5.0mm-4, B.Cu at (159.5, 100.0)
- added LED67: LED-RGB-CA, LEDs:LED_D5.0mm-4, B.Cu at (145.3, 154.8)
- added LED68: LED-RGB-CA, LEDs:LED_D5.0mm-4, B.Cu at (207.2, 83.3)
- added LED69: LED-RGB-CA, LEDs:LED_D5.0mm-4, B.Cu at (190.5, 138.1)
- added LED70: LED-RGB-CA, LEDs:LED_D5.0mm-4, B.Cu at (226.2, 83.3)
- added LED71: LED-RGB-CA, LEDs:LED_D5.0mm-4, B.Cu at (231.0, 169.1)
- added LED72: LED-RGB-CA, LEDs:LED_D5.0mm-4, B.Cu at (273.8, 100.0)
- added LED73: LED-RGB-CA, LEDs:LED_D5.0mm-4, B.Cu at (354.8, 145.3)
- added LED74: LED-RGB-CA, LEDs:LED_D5.0mm-4, B.Cu at (319.1, 81.0)
- added LED75: LED-RGB-CA, LEDs:LED_D5.0mm-4, B.Cu at (316.7, 171.4)
- added LED76: LED-RGB-CA, LEDs:LED_D5.0mm-4, B.Cu at (354.8, 109.5)
- added LED77: LED-RGB-CA, LEDs:LED_D5.0mm-4, B.Cu at (288.1, 154.8)
- added R1: 20kOhm, Resistors_SMD:R_0805_HandSoldering, B.Cu at (185.7, 166.7)
- added R2: 100kOhm, Resistors_SMD:R_0805_HandSoldering, B.Cu at (183.4, 166.7)
- added R3: 4.7kOhm, Resistors_SMD:R_0805_HandSoldering, B.Cu at (185.7, 159.5)
- added R5: 4.7kOhm, Resistors_SMD:R_0805_HandSoldering, B.Cu at (190.5, 159.5)
- added R6: 300, Resistors_SMD:R_0805_HandSoldering, F.Cu at (340.5, 97.6)
- added U1: IS31FL3731, Custom:IS31FL3731, B.Cu at (173.8, 161.9)
- HOLE1, HOLE2, HOLE3, HOLE4, HOLE5, HOLE6: value VAL** -> Mounting_Hole
- P1: value CONN_1 -> CONN_6; footprint Custom:CONN_1 -> Pin_Headers:Pin_Header_Straight_1x06_Pitch1.27mm; moved to B.Cu
- P2: value CONN_1 -> CONN_5; footprint Custom:CONN_1 -> Pin_Headers:Pin_Header_Straight_1x05_Pitch1.27mm; moved to B.Cu
- P3: value CONN_1 -> CONN_7X2; footprint Custom:CONN_1 -> Pin_Headers:Pin_Header_Straight_2x07_Pitch1.27mm
- P4: value CONN_1 -> CONN_4; footprint Custom:CONN_1 -> Pin_Headers:Pin_Header_Straight_1x04_Pitch1.27mm; moved to B.Cu
- R4: value 300 -> 4.7kOhm
- moved DB42 243.6 mm to (95.2, 145.3)
- moved DB54 212.8 mm to (85.7, 164.3)
- moved DB56 200.9 mm to (133.3, 164.3)
- moved DB59 166.7 mm to (300.0, 164.3)
- moved DB58 166.7 mm to (276.2, 164.3)
- moved R4 158.7 mm to (188.1, 159.5), turned to 270 degrees
- moved P1 124.2 mm to (352.4, 128.6)
- moved DB57 119.1 mm to (204.8, 164.3)
- moved DB60 119.1 mm to (323.9, 164.3)
- moved P2 101.1 mm to (323.9, 128.6)
- moved P4 64.3 mm to (161.9, 164.3)
- moved DB53 54.8 mm to (333.4, 145.3)
- moved DB52 38.1 mm to (297.7, 145.3)
- moved DB45 38.1 mm to (164.3, 145.3)
- moved DB46 38.1 mm to (183.4, 145.3)
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Connections:
- DB1 pad 1: LRow1 -> CA2
- DB1 pad 2: LCol1 -> CA1
- DB10 pad 1: LRow1 -> CA3
- DB10 pad 2: LCol10 -> CA2
- DB11 pad 1: LRow1 -> CA4
- DB11 pad 2: LCol11 -> CA2
- DB12 pad 1: LRow1 -> CA5
- DB12 pad 2: LCol12 -> CA2
- DB13 pad 1: LRow1 -> CA5
- DB13 pad 2: LCol13 -> CA2
- DB14 pad 1: LRow1 -> CA6
- DB14 pad 2: LCol14 -> CA2
- DB15 pad 1: LRow2 -> CA7
- DB15 pad 2: LCol1 -> CA2
- DB16 pad 1: LRow2 -> CA7
- DB16 pad 2: LCol2 -> CA2
- DB17 pad 1: LRow2 -> CA1
- DB17 pad 2: LCol3 -> CA3
- DB18 pad 1: LRow2 -> CA2
- DB18 pad 2: LCol4 -> CA3
- DB19 pad 1: LRow2 -> CA4
- DB19 pad 2: LCol5 -> CA3
- DB2 pad 1: LRow1 -> CA3
- DB2 pad 2: LCol2 -> CA1
- DB20 pad 1: LRow2 -> CA5
- DB20 pad 2: LCol6 -> CA3
- DB21 pad 1: LRow2 -> CA5
- DB21 pad 2: LCol7 -> CA3
- DB22 pad 1: LRow2 -> CA6
- DB22 pad 2: LCol8 -> CA3
- DB23 pad 1: LRow2 -> CA7
- DB23 pad 2: LCol9 -> CA3
- DB24 pad 1: LRow2 -> CA7
- DB24 pad 2: LCol10 -> CA3
- DB25 pad 1: LRow2 -> CA1
- DB25 pad 2: LCol11 -> CA4
- DB26 pad 1: LRow2 -> CA2
- DB26 pad 2: LCol12 -> CA4
- DB27 pad 1: LRow2 -> CA3
- DB27 pad 2: LCol13 -> CA4
- DB28 pad 1: LRow2 -> CA5
- DB28 pad 2: LCol14 -> CA4
- DB29 pad 1: LRow3 -> CA5
- DB29 pad 2: LCol1 -> CA4
- DB3 pad 1: LRow1 -> CA4
- DB3 pad 2: LCol3 -> CA1
- DB30 pad 1: LRow3 -> CA6
- DB30 pad 2: LCol2 -> CA4
- DB31 pad 1: LRow3 -> CA7
- DB31 pad 2: LCol3 -> CA4
- DB32 pad 1: LRow3 -> CA7
- DB32 pad 2: LCol4 -> CA4
- DB33 pad 1: LRow3 -> CA1
- DB33 pad 2: LCol5 -> CA5
- DB34 pad 1: LRow3 -> CA2
- DB34 pad 2: LCol6 -> CA5
- DB35 pad 1: LRow3 -> CA3
- DB35 pad 2: LCol7 -> CA5
- DB36 pad 1: LRow3 -> CA4
- DB36 pad 2: LCol8 -> CA5
- DB37 pad 1: LRow3 -> CA5
- DB37 pad 2: LCol9 -> CA5
- DB38 pad 1: LRow3 -> CA6
- DB38 pad 2: LCol10 -> CA5
- DB39 pad 1: LRow3 -> CA7
- DB39 pad 2: LCol11 -> CA5
- DB4 pad 1: LRow1 -> CA5
- DB4 pad 2: LCol4 -> CA1
- DB40 pad 1: LRow3 -> CA7
- DB40 pad 2: LCol12 -> CA5
- DB42 pad 1: LRow3 -> CA2
- DB42 pad 2: LCol14 -> CA5
- DB43 pad 1: LRow4 -> CA3
- DB43 pad 2: LCol1 -> CA5
- DB45 pad 1: LRow4 -> CA5
- DB45 pad 2: LCol3 -> CA5
- DB46 pad 1: LRow4 -> CA6
- DB46 pad 2: LCol4 -> CA5
- DB47 pad 1: LRow4 -> CA7
- DB47 pad 2: LCol5 -> CA5
- DB48 pad 1: LRow4 -> CA7
- DB48 pad 2: LCol6 -> CA5
- DB49 pad 1: LRow4 -> CA1
- DB49 pad 2: LCol7 -> CA6
- DB5 pad 1: LRow1 -> CA5
- DB5 pad 2: LCol5 -> CA1
- DB50 pad 1: LRow4 -> CA2
- DB50 pad 2: LCol8 -> CA6
- DB51 pad 1: LRow4 -> CA3
- DB51 pad 2: LCol9 -> CA6
- DB52 pad 1: LRow4 -> CA4
- DB52 pad 2: LCol10 -> CA6
- DB53 pad 1: LRow4 -> CA5
- DB53 pad 2: LCol11 -> CA6
- DB54 pad 1: LRow4 -> CA5
- DB54 pad 2: LCol12 -> CA6
- DB56 pad 1: LRow4 -> CA7
- DB56 pad 2: LCol14 -> CA6
- DB57 pad 1: LRow5 -> CA1
- DB57 pad 2: LCol1 -> CA7
- DB58 pad 1: LRow5 -> CA2
- DB58 pad 2: LCol2 -> CA7
- DB59 pad 1: LRow5 -> CA3
- DB59 pad 2: LCol3 -> CA7
- DB6 pad 1: LRow1 -> CA6
- DB6 pad 2: LCol6 -> CA1
- DB60 pad 1: LRow5 -> CA6
- DB60 pad 2: LCol6 -> CA7
- DB7 pad 1: LRow1 -> CA7
- DB7 pad 2: LCol7 -> CA1
- DB8 pad 1: LRow1 -> CA7
- DB8 pad 2: LCol8 -> CA1
- DB9 pad 1: LRow1 -> CA1
- DB9 pad 2: LCol9 -> CA2
- DC1 pad 1: Net-(DC1-Pad1) -> VCC
- DC1 pad 2: VCC -> Net-(DC1-Pad2)
- P1 pad 1: Col7 -> CAPS_LED
- P2 pad 1: Col6 -> Row5
- P3 pad 1: Col5 -> Col1
- P4 pad 1: Col4 -> Net-(P4-Pad1)
- R4 pad 1: Net-(DC1-Pad1) -> VCC
- R4 pad 2: CAPS_LED -> Net-(P4-Pad3)
Routing:
- net CA5: track 0.00 -> 598.9 mm, vias 0 -> 1
- net CB9: track 0.00 -> 591.1 mm, vias 0 -> 5
- net CB8: track 0.00 -> 568.0 mm, vias 0 -> 5
- net CA7: track 0.00 -> 551.7 mm, vias 0 -> 6
- net CA6: track 0.00 -> 546.6 mm, vias 0 -> 5
- net CA2: track 0.00 -> 521.8 mm, vias 0 -> 3
- net CB7: track 0.00 -> 475.3 mm, vias 0 -> 1
- net CA1: track 0.00 -> 472.8 mm, vias 0 -> 3
- net CA4: track 0.00 -> 472.2 mm, vias 0 -> 2
- net CB3: track 0.00 -> 472.0 mm, vias 0 -> 4
- net CA3: track 0.00 -> 459.4 mm, vias 0 -> 3
- net CB2: track 0.00 -> 442.8 mm, vias 0 -> 6
- net CB1: track 0.00 -> 423.0 mm, vias 0 -> 6
- net CB4: track 0.00 -> 317.9 mm, vias 0 -> 3
- net Row5: track 0.00 -> 316.8 mm, vias 0 -> 1
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Other:
- board text added: "PoliBoard - Ver 2 Designed by /u/ThePolikon"

Commit message: Add files via upload
Parts:
- moved LED75 40.5 mm to (357.2, 171.4), turned to 180 degrees
- moved LED74 38.2 mm to (357.2, 83.3), turned to 90 degrees
- moved C3 38.1 mm to (311.9, 150.0)
- moved C4 38.1 mm to (311.9, 147.6)
- moved C5 38.1 mm to (311.9, 145.3)
- moved C6 38.1 mm to (311.9, 142.9)
- moved C7 38.1 mm to (311.9, 140.5)
- moved LED64 33.4 mm to (76.2, 83.3), turned to 90 degrees
- moved LED66 33.1 mm to (131.0, 83.3)
- moved LED72 33.1 mm to (302.4, 83.3)
- moved LED69 31.3 mm to (195.3, 169.1)
- moved LED67 27.2 mm to (123.8, 171.4), turned to 90 degrees
- moved GND4 22.6 mm to (335.8, 154.8)
- moved LED65 21.6 mm to (78.6, 171.4), turned to 180 degrees
- moved C1 19.2 mm to (169.1, 164.3), turned to 270 degrees
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Connections:
- DB13 pad 1: CA5 -> CA6
- DB14 pad 1: CA6 -> CA7
- DB15 pad 1: CA7 -> CA8
- DB16 pad 1: CA7 -> CA8
- DB21 pad 1: CA5 -> CA6
- DB22 pad 1: CA6 -> CA7
- DB23 pad 1: CA7 -> CA8
- DB24 pad 1: CA7 -> CA8
- DB29 pad 1: CA5 -> CA6
- DB30 pad 1: CA6 -> CA7
- DB31 pad 1: CA7 -> CA8
- DB32 pad 1: CA7 -> CA8
- DB37 pad 1: CA5 -> CA6
- DB38 pad 1: CA6 -> CA7
- DB39 pad 1: CA7 -> CA8
- DB40 pad 1: CA7 -> CA8
- DB41 pad 2: CA5 -> CA6
- DB42 pad 2: CA5 -> CA6
- DB43 pad 2: CA5 -> CA6
- DB44 pad 2: CA5 -> CA6
- DB45 pad 2: CA5 -> CA6
- DB46 pad 1: CA6 -> CA7
- DB46 pad 2: CA5 -> CA6
- DB47 pad 1: CA7 -> CA8
- DB47 pad 2: CA5 -> CA6
- DB48 pad 1: CA7 -> CA8
- DB48 pad 2: CA5 -> CA6
- DB49 pad 2: CA6 -> CA7
- DB5 pad 1: CA5 -> CA6
- DB50 pad 2: CA6 -> CA7
- DB51 pad 2: CA6 -> CA7
- DB52 pad 2: CA6 -> CA7
- DB53 pad 2: CA6 -> CA7
- DB54 pad 1: CA5 -> CA6
- DB54 pad 2: CA6 -> CA7
- DB55 pad 1: CA7 -> CA8
- DB55 pad 2: CA6 -> CA7
- DB56 pad 1: CA7 -> CA8
- DB56 pad 2: CA6 -> CA7
- DB57 pad 2: CA7 -> CA8
- DB58 pad 2: CA7 -> CA8
- DB59 pad 2: CA7 -> CA8
- DB6 pad 1: CA6 -> CA7
- DB60 pad 2: CA7 -> CA8
- DB61 pad 2: CA7 -> CA8
- DB7 pad 1: CA7 -> CA8
- DB8 pad 1: CA7 -> CA8
- U1 pad 1: (no net) -> CA8
Routing:
- net CA8: track 0.00 -> 554.7 mm, vias 0 -> 3
- net CA5: track 598.9 -> 418.1 mm
- net CA7: track 551.7 -> 657.0 mm, vias 6 -> 2
- net CB4: track 317.9 -> 240.1 mm, vias 3 -> 2
- net Col10: track 143.6 -> 109.6 mm
- net CA6: track 546.6 -> 513.9 mm, vias 5 -> 1
- net Col1: track 260.7 -> 228.6 mm, vias 2 -> 0
- net CB7: track 475.3 -> 505.0 mm, vias 1 -> 3
- net CB9: track 591.1 -> 562.1 mm, vias 5 -> 0
- net CB3: track 472.0 -> 446.0 mm, vias 4 -> 1
- net Col11: track 145.5 -> 170.9 mm
- net CB8: track 568.0 -> 543.5 mm, vias 5 -> 2
- net CB1: track 423.0 -> 400.3 mm, vias 6 -> 0
- net Col14: track 236.5 -> 217.0 mm
- net CB6: track 269.0 -> 288.4 mm, vias 2 -> 1
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