File: Poliboard3.sch (KiCad schematic (older format))
At the start: 49 parts, among them P0 CONN_1, P1 CONN_1, P10 CONN_1, P11 CONN_1, P12 CONN_1, P13 CONN_1, P14 CONN_1, P15 CONN_1, P16 CONN_1, P17 CONN_1, P18 CONN_1, P19 CONN_1, P2 CONN_1, P20 CONN_1, P21 CONN_1, P22 CONN_1, P23 CONN_1, P24 CONN_1, P25 CONN_1, P26 CONN_1, P27 CONN_1, P28 CONN_1, P29 CONN_1, P3 CONN_1, P30 CONN_1, P31 CONN_1, P32 CONN_1, P33 CONN_1, P34 CONN_1, P35 CONN_1, P36 CONN_1, P37 CONN_1, P38 CONN_1, P39 CONN_1, P4 CONN_1, P40 CONN_1, P41 CONN_1, P42 CONN_1, P43 CONN_1, P5 CONN_1, P6 CONN_1, P7 CONN_1, P8 CONN_1, P9 CONN_1

Commit message: Add files via upload
Parts:
- removed P0, P1, P10, P11, P12, P13, P14, P15, P16, P17, P18, P19, P2, P20, P21, P22, P23, P24, P25, P26, P27, P28, P29, P3, P30, P31, P32, P33, P34, P35, P36, P37, P38, P39, P4, P40, P41, P42, P43, P5, P6, P7, P8, P9: CONN_1, Custom:CONN_1, symbol CONN_1
- added HOLE1, HOLE2, HOLE3, HOLE4: Mounting_Hole, Custom:HOLE1, symbol Mounting_Hole
- added HOLE5, HOLE6: Mounting_Hole, Custom:HOLE2, symbol Mounting_Hole
- added P1: CONN_6, Pin_Headers:Pin_Header_Straight_1x06_Pitch1.27mm, symbol CONN_6
- added P2, P4: CONN_5, Pin_Headers:Pin_Header_Straight_1x05_Pitch1.27mm, symbol CONN_5
- added P3, P5: CONN_7X2, Pin_Headers:Pin_Header_Straight_2x07_Pitch1.27mm, symbol CONN_7X2
Connections:
- net CAPS_LED: now also P1.1
- net Col1: now also P3.1 (P1)
- net Col10: now also P3.6 (P6)
- net Col11: now also P3.8 (P8)
- net Col12: now also P3.10
- net Col13: now also P3.12
- net Col14: now also P3.14
- net Col2: now also P3.3 (P3)
- net Col3: now also P3.5 (P5)
- net Col4: now also P3.7 (P7)
- net Col5: now also P3.9
- net Col6: now also P3.11
- net Col7: now also P3.13
- net Col8: now also P3.2 (P2)
- net Col9: now also P3.4 (P4)
- net GND: now also P1.3, P1.4, P1.5
- net LCol1: now also P5.1 (P1)
- net LCol10: now also P5.6 (P6)
- net LCol11: now also P5.8 (P8)
- net LCol12: now also P5.10
- net LCol13: now also P5.12
- net LCol14: now also P5.14
- net LCol2: now also P5.3 (P3)
- net LCol3: now also P5.5 (P5)
- net LCol4: now also P5.7 (P7)
- net LCol5: now also P5.9
- net LCol6: now also P5.11
- net LCol7: now also P5.13
- net LCol8: now also P5.2 (P2)
- net LCol9: now also P5.4 (P4)
- net LRow1: now also P4.1
- net LRow2: now also P4.2
- net LRow3: now also P4.3
- net LRow4: now also P4.4
- net LRow5: now also P4.5
- net Row1: now also P2.5
- net Row2: now also P2.4
- net Row3: now also P2.3
- net Row4: now also P2.2
- net Row5: now also P2.1
- net VCC: now also P1.2, P1.6

Commit message: Add files via upload
Parts:
- removed P4: CONN_5, Pin_Headers:Pin_Header_Straight_1x05_Pitch1.27mm, symbol CONN_5
- removed P5: CONN_7X2, Pin_Headers:Pin_Header_Straight_2x07_Pitch1.27mm, symbol CONN_7X2
- added C1: 1u, Capacitors_SMD:C_0805_HandSoldering, symbol C_Small
- added GND1, GND2, GND3, GND4, GND5: CONN_1, keyboard_parts:PIN_1, symbol CONN_1
- added P4: CONN_4, Pin_Headers:Pin_Header_Straight_1x04_Pitch1.27mm, symbol CONN_4
- added R1: 20kOhm, Resistors_SMD:R_0805_HandSoldering, symbol R
- added R2: 100kOhm, Resistors_SMD:R_0805_HandSoldering, symbol R
- added R3, R4, R5: 4.7kOhm, Resistors_SMD:R_0805_HandSoldering, symbol R
- added U1: IS31FL3731, Custom:IS31FL3731, symbol IS31FL3731
Connections:
- net GND: now also C1.2, GND1.1, GND2.1, GND3.1, GND4.1, GND5.1, R1.2, R2.2, U1.18 (AD), U1.5 (GND)
- net VCC: now also R3.1, R4.1, R5.1, U1.2 (VCC)
- new net: C1.1, U1.16 (C_FILT)
- new net: P4.4 (P4), R5.2, U1.19 (SDA)
- new net: P4.3 (P3), R4.2, U1.20 (SCL)
- new net: P4.1 (P1), R2.1, U1.3 (SDB)
- new net: P4.2 (P2), R3.2, U1.4 (INTB)
- new net: R1.1, U1.6 (R_EXT)
- new net CA1: U1.22 (C2)
- new net CA2: U1.23 (C3)
- new net CA3: U1.24 (C4)
- new net CA4: U1.25 (C5)
- new net CA5: U1.26 (C6)
- new net CA6: U1.27 (C7)
- new net CA7: U1.28 (C8)
- new net CB1: U1.7 (R9)
- new net CB2: U1.8 (R8)
- new net CB3: U1.9 (R7)
- new net CB4: U1.10 (R6)
- new net CB5: U1.11 (R5)
- new net CB6: U1.12 (R4)
- new net CB7: U1.13 (R3)
- new net CB8: U1.14 (R2)
- new net CB9: U1.15 (R1)
- no-connect marks 0 -> 3
Other:
- moved on the sheet: P1, P2, P3

Commit message: Add files via upload
Connections:
- net CA8: now reaches U1.1 (C9)
- no-connect marks 3 -> 2
Changed lines of the file:
@@
 Wire Wire Line
 	6000 1850 6450 1850
-NoConn ~ 6000 2150
 NoConn ~ 6000 1350
 $Comp
@@
 Wire Wire Line
 	6000 3100 6450 3100
+Text GLabel 6450 2150 2    60   Input ~ 0
+CA8
+Wire Wire Line
+	6000 2150 6450 2150
 $EndSCHEMATC

Commit message: Add files via upload
Parts:
- R1: value 20kOhm -> 18kOhm
Other:
- moved on the sheet: C3, C4, C5, C6, C7
Changed lines of the file:
@@
 L C_Small C3
 U 1 1 598F14B2
-P 700 1100
-F 0 "C3" H 710 1170 50  0000 L CNN
-F 1 "1u" H 710 1020 50  0000 L CNN
-F 2 "Capacitors_SMD:C_0805_HandSoldering" H 700 1100 50  0001 C CNN
-F 3 "" H 700 1100 50  0001 C CNN
-	1    700  1100
+P 5350 3800
+F 0 "C3" H 5360 3870 50  0000 L CNN
+F 1 "1u" H 5360 3720 50  0000 L CNN
+F 2 "Capacitors_SMD:C_0805_HandSoldering" H 5350 3800 50  0001 C CNN
+F 3 "" H 5350 3800 50  0001 C CNN
+	1    5350 3800
 	1    0    0    -1
 $EndComp
@@
 L C_Small C4
 U 1 1 598F1653
-P 900 1100
-F 0 "C4" H 910 1170 50  0000 L CNN
-F 1 "100n" H 910 1020 50  0000 L CNN
-F 2 "Capacitors_SMD:C_0805_HandSoldering" H 900 1100 50  0001 C CNN
-F 3 "" H 900 1100 50  0001 C CNN
-	1    900  1100
+P 5550 3800
+F 0 "C4" H 5560 3870 50  0000 L CNN
+F 1 "100n" H 5560 3720 50  0000 L CNN
+F 2 "Capacitors_SMD:C_0805_HandSoldering" H 5550 3800 50  0001 C CNN
+F 3 "" H 5550 3800 50  0001 C CNN
+	1    5550 3800
 	1    0    0    -1
 $EndComp
@@
 L C_Small C5
 U 1 1 598F1682
-P 1100 1100
-F 0 "C5" H 1110 1170 50  0000 L CNN
-F 1 "100n" H 1110 1020 50  0000 L CNN
-F 2 "Capacitors_SMD:C_0805_HandSoldering" H 1100 1100 50  0001 C CNN
-F 3 "" H 1100 1100 50  0001 C CNN
-	1    1100 1100
+P 5750 3800
+F 0 "C5" H 5760 3870 50  0000 L CNN
+F 1 "100n" H 5760 3720 50  0000 L CNN
+F 2 "Capacitors_SMD:C_0805_HandSoldering" H 5750 3800 50  0001 C CNN
+F 3 "" H 5750 3800 50  0001 C CNN
+	1    5750 3800
 	1    0    0    -1
 $EndComp
@@
 L C_Small C6
 U 1 1 598F16A5
-P 1300 1100
-F 0 "C6" H 1310 1170 50  0000 L CNN
-F 1 "100n" H 1310 1020 50  0000 L CNN
-F 2 "Capacitors_SMD:C_0805_HandSoldering" H 1300 1100 50  0001 C CNN
-F 3 "" H 1300 1100 50  0001 C CNN
-	1    1300 1100
+P 5950 3800
+F 0 "C6" H 5960 3870 50  0000 L CNN
+F 1 "100n" H 5960 3720 50  0000 L CNN
+F 2 "Capacitors_SMD:C_0805_HandSoldering" H 5950 3800 50  0001 C CNN
+F 3 "" H 5950 3800 50  0001 C CNN
+	1    5950 3800
 	1    0    0    -1
 $EndComp
@@
 L C_Small C7
 U 1 1 598F1761
-P 1500 1100
-F 0 "C7" H 1510 1170 50  0000 L CNN
-F 1 "100n" H 1510 1020 50  0000 L CNN
-F 2 "Capacitors_SMD:C_0805_HandSoldering" H 1500 1100 50  0001 C CNN
-F 3 "" H 1500 1100 50  0001 C CNN
-	1    1500 1100
+P 6150 3800
+F 0 "C7" H 6160 3870 50  0000 L CNN
+F 1 "100n" H 6160 3720 50  0000 L CNN
+F 2 "Capacitors_SMD:C_0805_HandSoldering" H 6150 3800 50  0001 C CNN
+F 3 "" H 6150 3800 50  0001 C CNN
+	1    6150 3800
 	1    0    0    -1
 $EndComp
@@
 L GND #PWR01
 U 1 1 598F1811
-P 700 1400
-F 0 "#PWR01" H 700 1150 50  0001 C CNN
-F 1 "GND" H 700 1250 50  0000 C CNN
-F 2 "" H 700 1400 50  0001 C CNN
-F 3 "" H 700 1400 50  0001 C CNN
-	1    700  1400
+P 5350 4100
+F 0 "#PWR01" H 5350 3850 50  0001 C CNN
+F 1 "GND" H 5350 3950 50  0000 C CNN
+F 2 "" H 5350 4100 50  0001 C CNN
+F 3 "" H 5350 4100 50  0001 C CNN
+	1    5350 4100
 	1    0    0    -1
 $EndComp
@@
 L VCC #PWR02
 U 1 1 598F1837
-P 700 800
-F 0 "#PWR02" H 700 650 50  0001 C CNN
-F 1 "VCC" H 700 950 50  0000 C CNN
-F 2 "" H 700 800 50  0001 C CNN
-F 3 "" H 700 800 50  0001 C CNN
-	1    700  800
+P 5350 3500
+F 0 "#PWR02" H 5350 3350 50  0001 C CNN
+F 1 "VCC" H 5350 3650 50  0000 C CNN
+F 2 "" H 5350 3500 50  0001 C CNN
+F 3 "" H 5350 3500 50  0001 C CNN
+	1    5350 3500
 	1    0    0    -1
 $EndComp
@@
 Col10
 Wire Wire Line
-	700  800  700  1000
-Wire Wire Line
-	700  1200 700  1400
-Wire Wire Line
-	700  1300 1500 1300
-Wire Wire Line
-	1500 1300 1500 1200
-Connection ~ 700  1300
-Wire Wire Line
-	1500 900  1500 1000
-Wire Wire Line
-	700  900  1500 900
-Connection ~ 700  900
-Wire Wire Line
-	900  900  900  1000
-Connection ~ 900  900
-Wire Wire Line
-	1100 900  1100 1000
-Connection ~ 1100 900
-Wire Wire Line
-	1300 900  1300 1000
-Connection ~ 1300 900
-Wire Wire Line
-	1300 1200 1300 1300
-Connection ~ 1300 1300
-Wire Wire Line
-	1100 1200 1100 1300
-Connection ~ 1100 1300
-Wire Wire Line
-	900  1200 900  1300
-Connection ~ 900  1300
+	5350 3500 5350 3700
+Wire Wire Line
+	5350 3900 5350 4100
+Wire Wire Line
+	5350 4000 6150 4000
+Wire Wire Line
+	6150 4000 6150 3900
+Connection ~ 5350 4000
+Wire Wire Line
+	6150 3600 6150 3700
+Wire Wire Line
+	5350 3600 6150 3600
+Connection ~ 5350 3600
+Wire Wire Line
+	5550 3600 5550 3700
+Connection ~ 5550 3600
+Wire Wire Line
+	5750 3600 5750 3700
+Connection ~ 5750 3600
+Wire Wire Line
+	5950 3600 5950 3700
+Connection ~ 5950 3600
+Wire Wire Line
+	5950 3900 5950 4000
+Connection ~ 5950 4000
+Wire Wire Line
+	5750 3900 5750 4000
+Connection ~ 5750 4000
+Wire Wire Line
+	5550 3900 5550 4000
+Connection ~ 5550 4000
 Wire Wire Line
 	1850 6350 2450 6350
@@
 P 4350 3050
 F 0 "R1" V 4430 3050 50  0000 C CNN
-F 1 "20kOhm" V 4350 3050 50  0000 C CNN
+F 1 "18kOhm" V 4350 3050 50  0000 C CNN
 F 2 "Resistors_SMD:R_0805_HandSoldering" H 4350 3050 60  0001 C CNN
 F 3 "" H 4350 3050 60  0001 C CNN
